File: kicad_analog_6bit/V3_16PIN/analog.kicad_pcb (KiCad board)
At the start: 2 copper layers, 50 x 23.2 mm, 30 parts, among them P1 Conn_02x05_Odd_Even, P2 Conn_01x04, P3 Conn_01x06, P4 Conn_01x02, P6 Conn_01x01, P7 Conn_01x01, U1 MAX9144, U2 MAX9144, U3 4066, U4 MAX5259EEE+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

Commit message: Analog V3 non-inverted 14 pin
Parts:
- R7, R8: value 100K -> 10K
- U3: value 4066 -> DG441xY; footprint Package_SO:SOIC-14_3.9x8.7mm_P1.27mm -> Package_SO:SOIC-16_3.9x9.9mm_P1.27mm
- moved U3 0.68 mm to (59.1, 49.2)
Connections:
- U3 pad 1: /SW_CLAMP -> /CLAMP
- U3 pad 11: /AGREEN -> /ABLUE
- U3 pad 12: /TERM_G -> /VCC
- U3 pad 13: /CLAMP -> /VCC
- U3 pad 14: /VCC -> /AGREEN
- U3 pad 2: /CLAMPLVL -> /SW_CLAMP
- U3 pad 3: /GND -> /CLAMPLVL
- U3 pad 4: /ARED -> /GND
- U3 pad 5: /TERM_RB -> /GND
- U3 pad 6: /TERM_RB -> /GND
- U3 pad 7: /GND -> /ARED
- U3 pad 8: /ABLUE -> /TERM_RB
- U3 pad 9: /GND -> /TERM_RB
Routing:
- net /TERM_RB: track 15.5 -> 32.1 mm
- net /GND: track 181.4 -> 168.8 mm, vias 13 -> 12
- net /AGREEN: track 54.0 -> 61.4 mm
- net /CLAMP: track 15.0 -> 21.4 mm
- net /TERM_G: track 16.8 -> 11.1 mm
- net /ABLUE: track 41.3 -> 46.4 mm
- net /VCC: track 113.1 -> 117.8 mm, vias 12 -> 13
- net /ARED: track 45.0 -> 42.6 mm
- net /GPIO22_STB: track 27.0 -> 25.9 mm
- net /REFRBUVHI: track 33.1 -> 33.8 mm
- net /REFRBUVLO: track 28.4 -> 29.0 mm
- net /GPIO1_CLK: track 35.9 -> 35.4 mm
