File: kicad_analog_6bit/Test/V3 - 14PIN TERM ONLY/analog.sch (KiCad schematic (older format))
At the start: 35 parts, among them P1 Conn_02x06_Odd_Even, P2 Conn_01x04, P3 Conn_01x06, P6 Conn_01x01, P7 Conn_01x01, U1 MAX9108, U2 MAX9108, U3 MAX4610, U4 MAX5259EEE+, U5 MCP1754S-3302xCB, U6 TS5A3159ADBVR, U7 MAX9108-Comparator

Commit message: V3 pcb plus some older alternatives
Parts:
- removed JP1, JP2: SolderJumper_3_Bridged12, Jumper:SolderJumper-3_P1.3mm_Bridged12_RoundedPad1.0x1.5mm, symbol Jumper:SolderJumper_3_Bridged12
- removed P1: Conn_02x06_Odd_Even, Connector_PinSocket_2.54mm:PinSocket_2x06_P2.54mm_Horizontal, symbol Connector_Generic:Conn_02x06_Odd_Even
- removed R10, R11, R9: 68R, Resistor_SMD:R_0805_2012Metric_Pad1.15x1.40mm_HandSolder, symbol Device:R_Small
- removed U6: TS5A3159ADBVR, Package_TO_SOT_SMD:SOT-23-6_Handsoldering, symbol Analog_Switch:TS5A3159ADBVR
- removed U7: MAX9108-Comparator, Package_SO:SOIC-14_3.9x8.7mm_P1.27mm, symbol analog-rescue:MAX9108-Comparator
- added C4: 10uF, Capacitor_SMD:C_0805_2012Metric_Pad1.15x1.40mm_HandSolder, symbol Device:C_Small
- added J1: Spare DAC, TestPoint:TestPoint_Pad_D1.0mm, symbol Connector_Generic:Conn_01x01
- added P1: Conn_02x05_Odd_Even, Connector_PinSocket_2.54mm:PinSocket_2x05_P2.54mm_Horizontal, symbol Connector_Generic:Conn_02x05_Odd_Even
- added P4: Conn_01x02, Connector_PinHeader_2.54mm:PinHeader_1x02_P2.54mm_Vertical, symbol Connector_Generic:Conn_01x02
- added R3: 1K, Resistor_SMD:R_0805_2012Metric_Pad1.15x1.40mm_HandSolder, symbol Device:R_Small
- added R5: 10K, Resistor_SMD:R_0805_2012Metric_Pad1.15x1.40mm_HandSolder, symbol Device:R_Small
- renumbered C6 to C1, C7 to C2, C8 to C3, C9 to C5, C2 to C6, C3 to C7, C4 to C8, C5 to C9, C1 to Cx1, R4 to R1, R3 to R4, R5 to R6, R6 to R7, R7 to R8, R8 to R9, R1 to Rx1
Connections:
- net labels added: SW_CLAMP, TERM_G, TERM_RB
- net labels removed: SGREEN, TERM, UV1, UV2, VCLAMP
- wire segments 224 -> 171
Other:
- moved on the sheet: C3, U1C, U2B, U2C
