File: kicad_analog_6bit/Test/V3 8BIT/analog.kicad_pcb (KiCad board)
At the start: 2 copper layers, 50 x 23.2 mm, 35 parts, among them P1 Conn_02x06_Odd_Even, P2 Conn_01x04, P3 Conn_01x06, P6 Conn_01x01, P7 Conn_01x01, U1 MAX9108, U2 MAX9108, U3 MAX4610, U4 MAX5259EEE+, U5 MCP1754S-3302xCB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

Commit message: V3 pcb plus some older alternatives
Parts:
- removed JP1, JP2: SolderJumper_3_Bridged12, Jumper:SolderJumper-3_P1.3mm_Bridged12_RoundedPad1.0x1.5mm
- R6, R7, R8: moved to B.Cu
- moved R8 11.2 mm to (75.0, 38.1), turned to 0 degrees
- moved C7 7.14 mm to (32.1, 47.5), turned to 0 degrees
- moved C6 6.37 mm to (35.9, 52.3), turned to 90 degrees
- moved R7 6.27 mm to (75.0, 40.1), turned to 0 degrees
- moved R2 5.87 mm to (69.4, 41.3), turned to 270 degrees
- moved R6 5.65 mm to (75.0, 42.3), turned to 0 degrees
- moved C5 5.64 mm to (35.9, 48.5), turned to 90 degrees
- moved U5 2.12 mm to (31.7, 50.8)
- moved D1 2.11 mm to (67.3, 35.1)
- moved U4 1.32 mm to (44.8, 51.4)
- moved C8 0.85 mm to (51.9, 52.4)
- moved R5 0.84 mm to (51.9, 48.1)
- moved C9 0.84 mm to (51.9, 50.3)
- moved U2 0.52 mm to (59.4, 39.6)
- moved R10 0.47 mm to (66.9, 50.5)
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Connections:
- P1 pad 11: /UV1 -> Net-(P1-Pad11)
- P1 pad 12: /UV2 -> Net-(P1-Pad12)
- U7 pad 13: /SPARE -> /CLAMPLVL
- U7 pad 2: /SPARE -> /CLAMPLVL
- U7 pad 6: /CLAMPLVL -> /SPARE
- U7 pad 9: /CLAMPLVL -> /SPARE
Routing:
- net /SPARE: track 42.2 -> 22.6 mm
- net /UV1: track 19.2 -> 0.00 mm, vias 1 -> 0
- net /ARED: track 80.0 -> 90.0 mm, vias 4 -> 2
- net /CLAMPLVL: track 38.3 -> 46.4 mm
- net /REFSYNC: track 21.6 -> 14.4 mm
- net /VCC: track 129.0 -> 135.8 mm, vias 13 -> 14
- net /UV2: track 6.64 -> 0.00 mm, vias 1 -> 0
- net /ABLUE: track 68.6 -> 75.0 mm
- net /REFGYSYNC: track 24.5 -> 19.0 mm
- net /GPIO1_CLK: track 32.4 -> 36.6 mm
- net Net-(U7-Pad8): track 3.85 -> 0.00 mm
- net Net-(U7-Pad1): track 3.84 -> 0.00 mm
- net /AGREEN: track 56.0 -> 59.6 mm
- net /GPIO0_DAT: track 38.0 -> 41.4 mm
- net /VCC_IN: track 10.6 -> 7.55 mm
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Other:
- board text added: "MAX5259 DAC Issue 3B ©2020 IanB"
- board text added: "Not Fitted"
- board text added: "Three level analog RGB/YUV & composite"
- board text removed: "Fit 10 way connector here"
- board text removed: "Fit for 12 way only"
- board text removed: "MAX5259 DAC Issue 3 ©2020 IanB"
- board text removed: "Three / Four level analog RGB/YUV & composite"
