File: kicad_analog_6bit/V3EIGHTold/analog.kicad_pcb (KiCad board)
At the start: 2 copper layers, 50 x 23.2 mm, 35 parts, among them P1 Conn_02x06_Odd_Even, P2 Conn_01x04, P3 Conn_01x06, P6 Conn_01x01, P7 Conn_01x01, U1 MAX9108, U2 MAX9108, U3 MAX4610, U4 MAX5259EEE+, U5 MCP1754S-3302xCB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

Commit message: V3 pcb plus some older alternatives
Parts:
- R10, R11, R9: moved to B.Cu
- moved R11 17.0 mm to (74.8, 38.0), turned to 0 degrees
- moved R8 14.2 mm to (67.0, 52.8), turned to 180 degrees
- moved R7 13.7 mm to (67.0, 50.8), turned to 180 degrees
- moved R10 13.4 mm to (74.8, 40.1), turned to 0 degrees
- moved R9 10.4 mm to (74.8, 42.2), turned to 0 degrees
- moved R6 7.50 mm to (67.0, 48.5), turned to 180 degrees
- moved R2 5.87 mm to (69.4, 41.3), turned to 270 degrees
- moved D1 2.11 mm to (67.3, 35.1)
- moved U2 0.52 mm to (59.4, 39.6)
- moved R1 0.20 mm to (54.2, 39.7)
- moved C1 0.14 mm to (52.1, 37.6)
Connections:
- R10 pad 2: Net-(R10-Pad2) -> /AGREEN
- R11 pad 2: Net-(R11-Pad2) -> /ARED
- R9 pad 2: Net-(R9-Pad2) -> /ABLUE
- U3 pad 11: Net-(R10-Pad2) -> /AGREEN
- U3 pad 4: Net-(R11-Pad2) -> /ARED
- U3 pad 8: Net-(R9-Pad2) -> /ABLUE
Routing:
- net /AGREEN: track 56.0 -> 73.8 mm, vias 2 -> 3
- net /ARED: track 80.0 -> 97.4 mm
- net /ABLUE: track 68.6 -> 81.3 mm, vias 1 -> 2
- net Net-(R10-Pad2): track 8.50 -> 0.00 mm
- net Net-(R11-Pad2): track 7.77 -> 0.00 mm
- net Net-(R9-Pad2): track 3.48 -> 0.00 mm
- net /VCC_IN: track 10.6 -> 7.55 mm
- net /ASYNC: track 25.7 -> 28.5 mm
- net /GND: track 194.2 -> 192.6 mm, vias 20 -> 17
- net /REFRBUVHI: track 31.1 -> 30.5 mm
- net /BBLUE: track 19.0 -> 18.5 mm
- net /RED: track 33.6 -> 34.1 mm
- net /BRED: track 25.3 -> 25.8 mm
- net /VCC: track 129.0 -> 129.5 mm, vias 13 -> 14
Other:
- board text added: "Cut shorting links"
- board text added: "if R9-R11 required"
